File: board/s100_enet.kicad_sch (KiCad schematic)
At the start: 34 parts, among them J1 FRAM socket, J2 SD Socket, J3 ClockSelect, P1 S100_MALE, SW1 SW_DIP_x08, U1 74LS10, U10 22V10, U11 74LS165, U12 74LS245, U13 74LS245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

Commit message: update schmatic
Connections:
- net DI0: now also U13.18 (B0)
- net DI1: now also U13.17 (B1)
- net DI2: now also U13.16 (B2)
- net DI3: now also U13.15 (B3)
- net DI4: now also U13.14 (B4)
- net DI5: now also U13.13 (B5)
- net DI6: now also U13.12 (B6)
- net DI7: now also U13.11 (B7)
- net DO0: now also U14.18 (B0)
- net DO1: now also U14.17 (B1)
- net DO2: now also U14.16 (B2)
- net DO3: now also U14.15 (B3)
- net DO4: now also U14.14 (B4)
- net DO5: now also U14.13 (B5)
- net DO6: now also U14.12 (B6)
- net DO7: now also U14.11 (B7)

Commit message: finish 22v10
Connections:
- net DIN is gone; now on net /IN_ENABLE: U13.19 (CE)
- net DOUT is gone; now on net /OUT_ENABLE: U14.19 (CE)
- net pWR* is gone; now on net pWR: P1.77 (pWR*)
- net sWO* is gone; now on net sWO: P1.97 (sWO*)
- net MWRT: now also U10.11 (I11)
- net pDBIN: now also U10.8 (I8)
- net sINP: now also U10.6 (I6)
- net sINTA: now also U10.3 (I3)
- net sM1: now also U10.2 (I2)
- net sMEMR: now also U10.9 (I9)
- net sOUT: now also U10.5 (I5)
- net /IORQ: now also U10.16 (O8)
- net /WR: now also U10.15 (O9)
- net SEL: now reaches U2.19 (P=R), U7.5 (E2)
- net SEL: now also U10.4 (I4)
- net sWO: now reaches U10.10 (I10)
- net /RD: now reaches U10.14 (O10)
- net /MREQ: now reaches U10.17 (O7)
- net /IN_ENABLE: now reaches U10.19 (O5)
- net /OUT_ENABLE: now reaches U10.21 (O3)
- net M1: now reaches U10.22 (O2)
- net pWR: now reaches U10.7 (I7)
- no-connect marks 56 -> 51
