File: board/new_enet/new_enet.kicad_pcb (KiCad board)
At the start: 2 copper layers, 254 x 134.6 mm, 36 parts, among them J1 FRAM socket, J2 SD Socket, J3 ClockSelect, P1 S100_MALE, SW1 SW_DIP_x08, U1 74LS10, U10 22V10, U11 74LS165, U12 74LS245, U13 74LS245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

Commit message: wip
Parts:
- J1: footprint Connector_PinHeader_1.00mm:PinHeader_1x08_P1.00mm_Horizontal -> Connector_PinHeader_2.54mm:PinHeader_1x08_P2.54mm_Vertical
- J2: footprint Connector_Harwin:Harwin_M20-89008xx_1x08_P2.54mm_Horizontal -> Connector_PinHeader_2.54mm:PinHeader_1x08_P2.54mm_Vertical
- moved J1 204.0 mm to (66.0, 53.3), turned to 90 degrees
- moved U8 85.1 mm to (130.8, 113.0)
- moved U2 81.8 mm to (113.0, 108.0)
- moved SW1 78.7 mm to (96.5, 109.2)
- moved J3 73.5 mm to (195.6, 134.6)
- moved U14 67.0 mm to (166.4, 110.5)
- moved U13 46.6 mm to (148.6, 110.5)
- moved U11 36.6 mm to (182.9, 114.3)
- moved U1 33.9 mm to (174.0, 88.9)
- moved U4 31.7 mm to (194.3, 91.4)
- moved J2 12.7 mm to (35.6, 53.3), turned to 90 degrees
- moved U12 5.68 mm to (73.7, 104.1), turned to 0 degrees
- moved U6 5.68 mm to (33.0, 110.8)
Routing:
- net BD0: track 0.00 -> 30.1 mm
- net +5V: track 0.00 -> 2.08 mm
