File: board/new_enet/new_enet.kicad_sch (KiCad schematic)
At the start: 34 parts, among them J1 FRAM socket, J2 SD Socket, J3 ClockSelect, P1 S100_MALE, SW1 SW_DIP_x08, U1 74LS10, U10 22V10, U11 74LS165, U12 74LS245, U13 74LS245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

Commit message: wip
Parts:
- J1: footprint Connector_PinHeader_1.00mm:PinHeader_1x08_P1.00mm_Horizontal -> Connector_PinHeader_2.54mm:PinHeader_1x08_P2.54mm_Vertical
- J2: footprint Connector_Harwin:Harwin_M20-89008xx_1x08_P2.54mm_Horizontal -> Connector_PinHeader_2.54mm:PinHeader_1x08_P2.54mm_Vertical
Changed lines of the file:
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@@
       (effects (font (size 1.27 1.27)) (justify right))
     )
-    (property "Footprint" "Connector_Harwin:Harwin_M20-89008xx_1x08_P2.54mm_Horizontal" (at 398.78 318.77 0)
+    (property "Footprint" "Connector_PinHeader_2.54mm:PinHeader_1x08_P2.54mm_Vertical" (at 398.78 318.77 0)
       (effects (font (size 1.27 1.27)) hide)
     )
@@
       (effects (font (size 1.27 1.27)) (justify right))
     )
-    (property "Footprint" "Connector_PinHeader_1.00mm:PinHeader_1x08_P1.00mm_Horizontal" (at 397.51 269.24 0)
-      (effects (font (size 1.27 1.27)) hide)
-    )
+    (property "Footprint" "Connector_PinHeader_2.54mm:PinHeader_1x08_P2.54mm_Vertical" (at 397.51 269.24 0)
+      (effects (font (size 1.27 1.27)) hide)
+    )
